File: XilinxFPGADevelopmentBoard.kicad_pcb (KiCad board)
At the start: 4 copper layers, 195 x 112 mm, 98 parts, among them J1 Conn_02x07_Odd_Even, J10 Conn_02x05_Odd_Even, J11 Conn_01x12_Pin, J12 Conn_02x09_Odd_Even, J2 DE15_Receptacle_HighDensity, J3 USB_B, J4 Conn_01x06, J5 Conn_01x12, J6 Conn_01x07_Socket, J7 Conn_01x10_Pin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

Commit message: Add files via upload
Other:
- board text added: "By Oriod Malo"
Changed lines of the file:
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@@
       (drillshape 0)
       (scaleselection 1)
-      (outputdirectory "/manufacturing")
+      (outputdirectory "C:/Users/CTS/Documents/KiCad/7.0/projects/XilinxFPGADevelopmentBoard/manufacturing")
     )
   )
@@
     (effects (font (size 3 3) (thickness 0.3)) (justify left bottom))
   )
+  (gr_text "By \nOriod Malo" (at 93.225 95.725) (layer "F.SilkS")
+    (effects (font (size 3 3) (thickness 0.4) italic) (justify left bottom))
+  )
   (gr_text "+3.3V" (at 73.8 86.35) (layer "F.SilkS")
